File: hdw/LED_Panel_Controller/PIC32MZ_Clocking.sch (KiCad schematic (older format))
At the start: 10 parts

Commit message: log's first
Parts:
- removed R?: 10k, Resistors_SMD:R_0402, symbol Custom_Library:R_Custom
- added C?: 0.1uF, Capacitors_SMD:C_0402, symbol Custom_Library:C_Custom
- added C?: 1nF, Capacitors_SMD:C_0402, symbol Custom_Library:C_Custom
- added C?: 10nF, Capacitors_SMD:C_0402, symbol Custom_Library:C_Custom
- added L?: 600R 0.5A, Inductors_SMD:L_0402, symbol Device:Ferrite_Bead
- added R?: 10k, Resistors_SMD:R_0402, symbol Custom_Library:R_Custom
- added R?: 100, Resistors_SMD:R_0402, symbol Custom_Library:R_Custom
- added X?: ECS-327KE, Custom Footprints Library:ECS-327KE, symbol Custom_Library:ECS-327KE
Connections:
- net PIC32MZ_POSC_EC_Enable is gone; now on an unnamed net: X?.1 (EN)
- net +3V3: now also L?.2
- net GND: now also C?.2, C?.2, C?.2, R?.2, X?.2 (GND)
- new net: R?.1, X?.3 (OUT)
- new net: C?.1, C?.1, C?.1, L?.1, X?.1 (EN), X?.4 (Vdd)
- new net PIC32MZ_SOSC_EC: R?.1, R?.2
