File: hdw/LED_Panel_Controller/LED_Panel_Controller.sch (KiCad schematic (older format))
At the start: 0 parts

Commit message: Many sch updates
Other:
- note added: "TODO:\n- Determine actual +12V current draw, reevaluate input protection circuit - 2A\n- Input EMI filter? - Drew\n- Determine image size, external flash size- 16,384 bytes\n- Determine +5V current draw, decide on converter - Drew - 3A\n- Determine +3.3V Current Draw, decide on converter - Drew\n- Remove high frequency PIC32MZ bypass caps - Drew\n- Figure out panel connectors - Drew\n* Figure out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"
- note removed: "TODO:\n* Determine actual +12V current draw, reevaluate input protection circuit\n* Determine image size, external flash size\n* Determine +5V current draw, decide on converter\n* Determine +3.3V Current Draw, decide on converter\n* Remove high frequency PIC32MZ bypass caps\n* Add PIC32MZ SOSC oscillator\n* Add +5V_USB capacitance/ESD?\n* Figure out panel connetors\n* Figure out panel level shift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"
Changed lines of the file:
@@
 33. Mechanical
 Text Notes 8660 6640 0    50   ~ 0
-TODO:\n* Determine actual +12V current draw, reevaluate input protection circuit\n* Determine image size, external flash size\n* Determine +5V current draw, decide on converter\n* Determine +3.3V Current Draw, decide on converter\n* Remove high frequency PIC32MZ bypass caps\n* Add PIC32MZ SOSC oscillator\n* Add +5V_USB capacitance/ESD?\n* Figure out panel connetors\n* Figure out panel level shifting\n* Figure out SPI flash circuit\n* Figure out screen modes/mode LEDs\n* Draw SD card sheet\n* Draw WiFi module sheet\n* Draw I2C boost sheet with LTC1694\n* Determine what will be configurable, add hardstraps\n* What will pushbuttons do?\n* What PIC32MZ SKU will we use? Should be highest memory + speed\n* Change PGOOD LEDs sheet to use +3.3V_PGL global power symbol
+TODO:\n- Determine actual +12V current draw, reevaluate input protection circuit - 2A\n- Input EMI filter? - Drew\n- Determine image size, external flash size- 16,384 bytes\n- Determine +5V current draw, decide on converter - Drew - 3A\n- Determine +3.3V Current Draw, decide on converter - Drew\n- Remove high frequency PIC32MZ bypass caps - Drew\n- Figure out panel connectors - Drew\n* Figure out panel level shifting - Logan\n- Figure out SPI flash circuit - Drew\n* Figure out screen modes/mode LEDs\n- Draw SD card sheet - Logan\n* Draw WiFi module sheet\n- Draw I2C boost sheet with LTC1694 - Drew\n* Determine what will be configurable, add hardstraps\n* What will pushbuttons do?\n* What PIC32MZ SKU will we use? Should be highest memory + speed - Drew\n- Change PGOOD LEDs sheet to use +3.3V_PGL global power symbol - Drew\n* Add USB Telemetry sheet\n
 $EndSCHEMATC

Commit message: reworked some USB stuff
Changed lines of the file:
@@
 $Descr A 11000 8500
 encoding utf-8
-Sheet 1 33
+Sheet 1 34
 Title ""
 Date "2020-09-08"
@@
 Text Notes 8660 6640 0    50   ~ 0
 TODO:\n- Determine actual +12V current draw, reevaluate input protection circuit - 2A\n- Input EMI filter? - Drew\n- Determine image size, external flash size- 16,384 bytes\n- Determine +5V current draw, decide on converter - Drew - 3A\n- Determine +3.3V Current Draw, decide on converter - Drew\n- Remove high frequency PIC32MZ bypass caps - Drew\n- Figure out panel connectors - Drew\n* Figure out panel level shifting - Logan\n- Figure out SPI flash circuit - Drew\n* Figure out screen modes/mode LEDs\n- Draw SD card sheet - Logan\n* Draw WiFi module sheet\n- Draw I2C boost sheet with LTC1694 - Drew\n* Determine what will be configurable, add hardstraps\n* What will pushbuttons do?\n* What PIC32MZ SKU will we use? Should be highest memory + speed - Drew\n- Change PGOOD LEDs sheet to use +3.3V_PGL global power symbol - Drew\n* Add USB Telemetry sheet\n
+$Sheet
+S 7030 5770 500  150
+U 5F7B4289
+F0 "USB Telemetry" 50
+F1 "USB_Telemetry.sch" 50
+$EndSheet
 $EndSCHEMATC
