File: hdw/LED_Panel_Controller/PGOOD_LEDs.sch (KiCad schematic (older format))
At the start: 14 parts

Commit message: Many sch updates
Parts:
- removed C? (x2): 0.1uF, Capacitors_SMD:C_0402, symbol Custom_Library:C_Custom
- removed C?: 10uF, Capacitors_SMD:C_0402, symbol Custom_Library:C_Custom
- removed D?: Green, LEDs:LED_0402, symbol Device:LED
- removed R?: 1k, Resistors_SMD:R_0402, symbol Custom_Library:R_Custom
- removed U? (x3): 74LVC1G06, TO_SOT_Packages_SMD:SOT-353_SC-70-5, symbol Custom_Library:74LVC1G06_Power
- removed U?: TPS71530, Package_TO_SOT_SMD:SOT-353_SC-70-5, symbol Regulator_Linear:TPS71530__SC70
- added C? (x4): 0.1uF, Capacitors_SMD:C_0603, symbol Custom_Library:C_Custom
- added C? (x2): 4.7uF, Capacitors_SMD:C_0805, symbol Custom_Library:C_Custom
- added D? (x2): Green, LEDs:LED_0603, symbol Device:LED
- added D?: Red, LEDs:LED_0603, symbol Device:LED
- added Q?: BSS214NW, Package_TO_SOT_SMD:SOT-323_SC-70, symbol Transistor_FET:BSS214NW
- added R? (x3): 1k, Resistors_SMD:R_0603, symbol Custom_Library:R_Custom
- added R? (x2): 10k, Resistors_SMD:R_0603, symbol Custom_Library:R_Custom
- added R?: 10, Resistors_SMD:R_0603, symbol Custom_Library:R_Custom
- added U? (x4): 74LVC1G06, TO_SOT_Packages_SMD:SOT-353_SC-70-5, symbol Custom_Library:74LVC1G06_Power
- added U?: LP2985-3.3, Package_TO_SOT_SMD:SOT-23-5, symbol Regulator_Linear:LP2985-3.3
- added U?: 74LVC1G07, TO_SOT_Packages_SMD:SOT-353_SC-70-5, symbol Custom_Library:74LVC1G07_Power
- C?: footprint Capacitors_SMD:C_0402 -> Capacitors_SMD:C_0603; Digi-Key PN (none) -> 399-7845-1-ND; display_footprint 0402 -> 0603
- D? (x2): footprint LEDs:LED_0402 -> LEDs:LED_0603; Digi-Key PN 1497-1219-1-ND -> 754-1121-1-ND
- R? (x2): footprint Resistors_SMD:R_0402 -> Resistors_SMD:R_0603; Digi-Key PN (none) -> 311-1.00KHRCT-ND; Wattage 1/16W -> 1/10W; display_footprint 0402 -> 0603
Connections:
- net labels added: +3.3V_PGL, POS3P3_PGL_SHDN, POS5_USB_PGOOD, VBAT_PGOOD
- wire segments 15 -> 22
- no-connect marks 0 -> 1
Other:
- moved on the sheet: C?, D?, R?
