File: hdw/LED_Panel_Controller/POS5_Power_Supply.sch (KiCad schematic (older format))
At the start: 0 parts

Commit message: Many sch updates
Parts:
- added C?: 10uF, Capacitors_SMD:C_1206, symbol Custom_Library:C_Custom
- added C?: 100uF, symbol Custom_Library:C_Custom
- added C? (x2): 0.1uF, Capacitors_SMD:C_0402, symbol Custom_Library:C_Custom
- added C?: 10nF, Capacitors_SMD:C_0402, symbol Custom_Library:C_Custom
- added C?: 10uF, Capacitors_SMD:C_0402, symbol Custom_Library:C_Custom
- added D?: BAT48JFILM, Diode_SMD:D_SOD-323, symbol Diode:BAT48JFILM
- added L?: 2.2uH, symbol Custom_Library:L_Custom
- added Q?: ZXMS6004FFTA, Package_TO_SOT_SMD:SOT-23, symbol Custom_Library:ZXMS6004FFTA
- added Q?: BSS214NW, Package_TO_SOT_SMD:SOT-323_SC-70, symbol Transistor_FET:BSS214NW
- added R?: 953k, Resistors_SMD:R_0402, symbol Custom_Library:R_Custom
- added R?: 0.02, Resistors_SMD:R_0612, symbol Custom_Library:R_Custom
- added R? (x3): 10k, Resistors_SMD:R_0402, symbol Custom_Library:R_Custom
- added R?: 180k, Resistors_SMD:R_0402, symbol Custom_Library:R_Custom
- added R? (x2): 10, Resistors_SMD:R_0402, symbol Custom_Library:R_Custom
- added TP?: TP, Custom Footprints Library:Test_Point, symbol Custom_Library:TP
- added U?: TPS62130, Package_DFN_QFN:QFN-16-1EP_3x3mm_P0.5mm_EP1.8x1.8mm, symbol Custom_Library:TPS62130
Connections:
- new net: C?.1, L?.2, R?.1, R?.2
- new net: R?.1, R?.2, U?.5 (FB)
- new net: C?.1, U?.9 (SS/TR)
- new net: Q?.1 (G), Q?.3 (D), R?.2
- new net: C?.1, D?.1 (K), R?.1
- new net: L?.1, U?.1 (SW), U?.2 (SW), U?.3 (SW)
- new net +12V: C?.1, C?.1, U?.10 (AVIN), U?.11 (PVIN), U?.12 (PVIN)
- new net +3V3: D?.2 (A), R?.1
- new net +5V: C?.1, R?.1, R?.2, R?.2, TP?.1 (TP), U?.14 (VOS)
- new net GND: C?.2, C?.2, C?.2, C?.2, C?.2, C?.2, Q?.2 (S), Q?.2 (S), R?.2, R?.2, U?.15 (PGND), U?.16 (PGND), U?.17 (EP), U?.6 (AGND), U?.7 (FSW), U?.8 (DEF)
- new net POS5_PGOOD: R?.2, U?.4 (PG)
- new net POS5_RUN: Q?.1 (G), R?.1, U?.13 (EN)
- new net POS5_SNS_OUT+: R?.1
- new net POS5_SNS_OUT-: R?.1
