File: hdw/LED_Panel_Controller/SPI_Flash_0.sch (KiCad schematic (older format))
At the start: 0 parts

Commit message: Many sch updates
Parts:
- added C? (x2): 0.1uF, Capacitors_SMD:C_0603, symbol Custom_Library:C_Custom
- added D?: Green, LEDs:LED_0603, symbol Device:LED
- added R? (x4): 10k, Resistors_SMD:R_0603, symbol Custom_Library:R_Custom
- added R? (x4): 10, symbol Custom_Library:R_Custom
- added R?: 1k, Resistors_SMD:R_0603, symbol Custom_Library:R_Custom
- added U?: 74LVC1G07, TO_SOT_Packages_SMD:SOT-353_SC-70-5, symbol Custom_Library:74LVC1G07_Power
- added U?: SST25VF080B-50-4I-S2AF, Package_SO:SOIC-8_5.275x5.275mm_P1.27mm, symbol Memory_Flash:SST25VF080B-50-4x-S2Ax
Connections:
- new net: R?.1, R?.1, U?.5 (SI)
- new net: R?.1, R?.2, U?.1 (~CE)
- new net: R?.1, R?.1, U?.2 (SO)
- new net: D?.1 (K), U?.4
- new net: D?.2 (A), R?.2
- new net: R?.1, R?.1, U?.6 (SCK)
- new net +3V3: C?.1, C?.1, R?.1, R?.1, U?.3 (~WP~), U?.5 (VCC), U?.7 (~HOLD~), U?.8 (VDD)
- new net FLASH_SPI_MISO: R?.2
- new net FLASH_SPI_MOSI: R?.2
- new net FLASH_SPI_SCK: R?.2
- new net GND: C?.2, C?.2, R?.2, R?.2, R?.2, U?.3 (GND), U?.4 (VSS)
- new net ~FLASH_SPI_CE1: R?.2, U?.2
