File: hdw/LED_Panel_Controller/WiFi_Module.sch (KiCad schematic (older format))
At the start: 0 parts

Commit message: lots of schematic progress
Parts:
- added C?: 10nF, symbol Custom_Library:C_Custom
- added C? (x5): 10uF, Capacitors_SMD:C_0402, symbol Custom_Library:C_Custom
- added J?: WIFI_I2C, symbol Connector_Generic:Conn_01x03
- added R? (x10): 10k, Resistors_SMD:R_0402, symbol Custom_Library:R_Custom
- added R? (x7): 10, Resistors_SMD:R_0402, symbol Custom_Library:R_Custom
- added R?: 1M, Resistors_SMD:R_0402, symbol Custom_Library:R_Custom
- added TP?: TP_Pad, Custom Footprints Library:Test_Point, symbol Custom_Library:TP_Pad
- added U?: ATWINC1500-MR210PB, symbol Custom_Library:ATWINC1500-MR210PB
Connections:
- new net: R?.2, U?.10 (SPI_CFG)
- new net: R?.1, R?.1, U?.13 (IRQN)
- new net: R?.1, R?.1, U?.15 (SPI_RXD)
- new net: R?.1, R?.2, U?.16 (~SPI_SSN~)
- new net: R?.1, R?.1, U?.17 (SPI_TXD)
- new net: R?.1, R?.1, U?.18 (SPI_SCK)
- new net: J?.1 (Pin_1), R?.2, U?.2 (I2C_SCL)
- new net: R?.1, R?.1, U?.22 (CHIP_EN)
- new net: J?.2 (Pin_2), R?.2, U?.3 (I2C_SDA)
- new net: R?.1, R?.1, U?.4 (~RESET_N~)
- new net +3V3: C?.1, C?.1, C?.1, C?.1, R?.1, R?.1, R?.1, R?.1, U?.20 (VBATT), U?.23 (VDDIO)
- new net GND: C?.2, C?.2, C?.2, C?.2, C?.2, C?.2, J?.3 (Pin_3), R?.2, R?.2, R?.2, R?.2, R?.2, R?.2, R?.2, U?.29 (PADDLE_GND), U?.9 (GND)
- new net WIFI_CHIP_EN: R?.2
- new net WIFI_IRQN: R?.2
- new net WIFI_SPI_MISO: R?.2
- new net WIFI_SPI_MOSI: R?.2
- new net WIFI_SPI_SCK: R?.2
- new net WIFI_UART_RX: U?.19 (UART_RXD)
- new net WIFI_UART_TX: U?.14 (UART_TXD)
- new net WIFI_VCORE: C?.1, C?.1, TP?.1 (TP), U?.24 (1P3V_TP)
- new net WIFI_WAKE: R?.1, U?.11 (WAKE)
- new net ~WIFI_RESET: R?.2
- new net ~WIFI_SPI_SS: R?.2

Commit message: made a lot more schematic progress
Parts:
- removed C? (x3): 10uF, Capacitors_SMD:C_0402, symbol Custom_Library:C_Custom
- added C? (x3): 10uF, Capacitors_SMD:C_0402, symbol Custom_Library:C_Custom
- C? (x3), U?: Configuration (none) -> WIFI
Connections:
- net +3V3: now also C?.1, C?.1, C?.1
- net GND: now also C?.2, C?.2, C?.2
Changed lines of the file:
@@
 F 3 "https://ww1.microchip.com/downloads/en/DeviceDoc/ATWINC15x0-MR210xB-IEEE-802.11-b-g-n-SmartConnect-IoT-Module-Data-Sheet-DS70005304C.pdf" H 6250 3700 50  0001 L BNN
 F 4 "ATWINC1500-MR210PB-ND" H 6250 3700 50  0001 C CNN "Digi-Key PN"
+F 5 "WIFI" H 6250 2140 50  0000 C CNN "Configuration"
 	1    6250 3700
 	1    0    0    -1
@@
 F 5 "50V" H 7180 3530 50  0000 R CNN "Voltage"
 F 6 "X7R" H 7180 3430 50  0000 R CNN "Dielectric"
-F 7 "" H 7755 4030 60  0001 C CNN "Digi-Key PN"
+F 7 "WIFI" H 7180 3710 50  0000 R CNN "Configuration"
 	1    7330 3530
 	1    0    0    -1
@@
 F 6 "X5R" H 7930 3430 50  0000 R CNN "Dielectric"
 F 7 "490-13211-1-ND" H 8080 3530 50  0001 C CNN "Digi-Key PN"
+F 8 "WIFI" H 7930 3710 50  0000 R CNN "Configuration"
 	1    8080 3530
 	1    0    0    -1
@@
 Text Label 7480 3300 0    50   ~ 0
 WIFI_VCORE
-$Comp
-L Custom_Library:R_Custom R?
-U 1 1 5FF2C483
-P 7330 2930
-AR Path="/5D6B2673/5FF2C483" Ref="R?"  Part="1"
-AR Path="/5D6C0D23/5FF2C483" Ref="R?"  Part="1"
-AR Path="/5D77A516/5FF2C483" Ref="R?"  Part="1"
-AR Path="/5E939CFF/5FF2C483" Ref="R?"  Part="1"
-AR Path="/5F581B41/5FF2C483" Ref="R?"  Part="1"
-AR Path="/5F582E44/5FF2C483" Ref="R?"  Part="1"
-F 0 "R?" H 7240 2930 50  0000 R CNN
-F 1 "10k" V 7330 2860 50  0000 L CNN
-F 2 "Resistors_SMD:R_0402" H 7330 2930 50  0001 C CNN
-F 3 "" H 7330 2930 50  0001 C CNN
-F 4 "0402" H 7430 3000 50  0000 L CNN "display_footprint"
-F 5 "1%" H 7430 2900 50  0000 L CNN "Tolerance"
-F 6 "1/16W" H 7430 2800 50  0000 L CNN "Wattage"
-F 7 "" H 7630 3330 60  0001 C CNN "Digi-Key PN"
-	1    7330 2930
-	-1   0    0    -1
-$EndComp
 $Comp
 L power:GND #PWR?
@@
 	2380 4800 2300 4800
 $Comp
-L Custom_Library:C_Custom C?
-U 1 1 5FF8CED8
-P 6710 1610
-AR Path="/5CB7718D/5FF8CED8" Ref="C?"  Part="1"
-AR Path="/5E0DC082/5FF8CED8" Ref="C?"  Part="1"
-AR Path="/5E0F9110/5FF8CED8" Ref="C?"  Part="1"
-AR Path="/5A557C58/5FF8CED8" Ref="C?"  Part="1"
-AR Path="/5CB25152/5FF8CED8" Ref="C?"  Part="1"
-AR Path="/5E697934/5FF8CED8" Ref="C?"  Part="1"
-AR Path="/5EAE2F02/5FF8CED8" Ref="C?"  Part="1"
-AR Path="/5EAE3021/5FF8CED8" Ref="C?"  Part="1"
-AR Path="/5EAE2D8A/5FF8CED8" Ref="C?"  Part="1"
-AR Path="/5F581B64/5FF8CED8" Ref="C?"  Part="1"
-AR Path="/5F582E44/5FF8CED8" Ref="C?"  Part="1"
-F 0 "C?" H 6735 1710 50  0000 L CNN
-F 1 "10uF" H 6735 1510 50  0000 L CNN
-F 2 "Capacitors_SMD:C_0402" H 6748 1460 50  0001 C CNN
-F 3 "" H 6735 1710 50  0001 C CNN
-F 4 "0402" H 6560 1710 50  0000 R CNN "display_footprint"
-F 5 "6.3V" H 6560 1610 50  0000 R CNN "Voltage"
-F 6 "X5R" H 6560 1510 50  0000 R CNN "Dielectric"
-F 7 "490-13211-1-ND" H 6710 1610 50  0001 C CNN "Digi-Key PN"
-	1    6710 1610
-	1    0    0    -1
-$EndComp
-$Comp
 L power:GND #PWR?
 U 1 1 5FF8DBDF
@@
 F 3 "" H 6710 1460 50  0001 C CNN
 	1    6710 1460
-	1    0    0    -1
-$EndComp
-$Comp
-L Custom_Library:C_Custom C?
-U 1 1 5FF8E14F
-P 7410 1610
-AR Path="/5CB7718D/5FF8E14F" Ref="C?"  Part="1"
-AR Path="/5E0DC082/5FF8E14F" Ref="C?"  Part="1"
-AR Path="/5E0F9110/5FF8E14F" Ref="C?"  Part="1"
-AR Path="/5A557C58/5FF8E14F" Ref="C?"  Part="1"
-AR Path="/5CB25152/5FF8E14F" Ref="C?"  Part="1"
-AR Path="/5E697934/5FF8E14F" Ref="C?"  Part="1"
-AR Path="/5EAE2F02/5FF8E14F" Ref="C?"  Part="1"
-AR Path="/5EAE3021/5FF8E14F" Ref="C?"  Part="1"
-AR Path="/5EAE2D8A/5FF8E14F" Ref="C?"  Part="1"
-AR Path="/5F581B64/5FF8E14F" Ref="C?"  Part="1"
-AR Path="/5F582E44/5FF8E14F" Ref="C?"  Part="1"
-F 0 "C?" H 7435 1710 50  0000 L CNN
-F 1 "10uF" H 7435 1510 50  0000 L CNN
-F 2 "Capacitors_SMD:C_0402" H 7448 1460 50  0001 C CNN
-F 3 "" H 7435 1710 50  0001 C CNN
-F 4 "0402" H 7260 1710 50  0000 R CNN "display_footprint"
-F 5 "6.3V" H 7260 1610 50  0000 R CNN "Voltage"
-F 6 "X5R" H 7260 1510 50  0000 R CNN "Dielectric"
-F 7 "490-13211-1-ND" H 7410 1610 50  0001 C CNN "Digi-Key PN"
-	1    7410 1610
 	1    0    0    -1
 $EndComp
@@
 F 6 "X5R" H 5160 1510 50  0000 R CNN "Dielectric"
 F 7 "490-13211-1-ND" H 5310 1610 50  0001 C CNN "Digi-Key PN"
+F 8 "WIFI" H 5150 1780 50  0000 R CNN "Configuration"
 	1    5310 1610
 	1    0    0    -1
@@
 $EndComp
 $Comp
+L power:GND #PWR?
+U 1 1 5FF91EC9
+P 6010 1760
+F 0 "#PWR?" H 6010 1510 50  0001 C CNN
+F 1 "GND" H 6010 1610 50  0000 C CNN
+F 2 "" H 6010 1760 50  0001 C CNN
+F 3 "" H 6010 1760 50  0001 C CNN
+	1    6010 1760
+	1    0    0    -1
+$EndComp
+$Comp
+L power:+3.3V #PWR?
+U 1 1 5FF91ED3
+P 6010 1460
+F 0 "#PWR?" H 6010 1310 50  0001 C CNN
+F 1 "+3.3V" H 6010 1600 50  0000 C CNN
+F 2 "" H 6010 1460 50  0001 C CNN
+F 3 "" H 6010 1460 50  0001 C CNN
+	1    6010 1460
+	1    0    0    -1
+$EndComp
+$Comp
 L Custom_Library:C_Custom C?
-U 1 1 5FF91EBF
+U 1 1 6020EF8E
 P 6010 1610
-AR Path="/5CB7718D/5FF91EBF" Ref="C?"  Part="1"
-AR Path="/5E0DC082/5FF91EBF" Ref="C?"  Part="1"
-AR Path="/5E0F9110/5FF91EBF" Ref="C?"  Part="1"
-AR Path="/5A557C58/5FF91EBF" Ref="C?"  Part="1"
-AR Path="/5CB25152/5FF91EBF" Ref="C?"  Part="1"
-AR Path="/5E697934/5FF91EBF" Ref="C?"  Part="1"
-AR Path="/5EAE2F02/5FF91EBF" Ref="C?"  Part="1"
-AR Path="/5EAE3021/5FF91EBF" Ref="C?"  Part="1"
-AR Path="/5EAE2D8A/5FF91EBF" Ref="C?"  Part="1"
-AR Path="/5F581B64/5FF91EBF" Ref="C?"  Part="1"
-AR Path="/5F582E44/5FF91EBF" Ref="C?"  Part="1"
+AR Path="/5CB7718D/6020EF8E" Ref="C?"  Part="1"
+AR Path="/5E0DC082/6020EF8E" Ref="C?"  Part="1"
+AR Path="/5E0F9110/6020EF8E" Ref="C?"  Part="1"
+AR Path="/5A557C58/6020EF8E" Ref="C?"  Part="1"
+AR Path="/5CB25152/6020EF8E" Ref="C?"  Part="1"
+AR Path="/5E697934/6020EF8E" Ref="C?"  Part="1"
+AR Path="/5EAE2F02/6020EF8E" Ref="C?"  Part="1"
+AR Path="/5EAE3021/6020EF8E" Ref="C?"  Part="1"
+AR Path="/5EAE2D8A/6020EF8E" Ref="C?"  Part="1"
+AR Path="/5F581B64/6020EF8E" Ref="C?"  Part="1"
+AR Path="/5F582E44/6020EF8E" Ref="C?"  Part="1"
 F 0 "C?" H 6035 1710 50  0000 L CNN
 F 1 "10uF" H 6035 1510 50  0000 L CNN
@@
 F 6 "X5R" H 5860 1510 50  0000 R CNN "Dielectric"
 F 7 "490-13211-1-ND" H 6010 1610 50  0001 C CNN "Digi-Key PN"
+F 8 "WIFI" H 5850 1780 50  0000 R CNN "Configuration"
 	1    6010 1610
 	1    0    0    -1
 $EndComp
 $Comp
-L power:GND #PWR?
-U 1 1 5FF91EC9
-P 6010 1760
-F 0 "#PWR?" H 6010 1510 50  0001 C CNN
-F 1 "GND" H 6010 1610 50  0000 C CNN
-F 2 "" H 6010 1760 50  0001 C CNN
-F 3 "" H 6010 1760 50  0001 C CNN
-	1    6010 1760
-	1    0    0    -1
-$EndComp
-$Comp
-L power:+3.3V #PWR?
-U 1 1 5FF91ED3
-P 6010 1460
-F 0 "#PWR?" H 6010 1310 50  0001 C CNN
-F 1 "+3.3V" H 6010 1600 50  0000 C CNN
-F 2 "" H 6010 1460 50  0001 C CNN
-F 3 "" H 6010 1460 50  0001 C CNN
-	1    6010 1460
-	1    0    0    -1
+L Custom_Library:C_Custom C?
+U 1 1 6020F45D
+P 6710 1610
+AR Path="/5CB7718D/6020F45D" Ref="C?"  Part="1"
+AR Path="/5E0DC082/6020F45D" Ref="C?"  Part="1"
+AR Path="/5E0F9110/6020F45D" Ref="C?"  Part="1"
+AR Path="/5A557C58/6020F45D" Ref="C?"  Part="1"
+AR Path="/5CB25152/6020F45D" Ref="C?"  Part="1"
+AR Path="/5E697934/6020F45D" Ref="C?"  Part="1"
+AR Path="/5EAE2F02/6020F45D" Ref="C?"  Part="1"
+AR Path="/5EAE3021/6020F45D" Ref="C?"  Part="1"
+AR Path="/5EAE2D8A/6020F45D" Ref="C?"  Part="1"
+AR Path="/5F581B64/6020F45D" Ref="C?"  Part="1"
+AR Path="/5F582E44/6020F45D" Ref="C?"  Part="1"
+F 0 "C?" H 6735 1710 50  0000 L CNN
+F 1 "10uF" H 6735 1510 50  0000 L CNN
+F 2 "Capacitors_SMD:C_0402" H 6748 1460 50  0001 C CNN
+F 3 "" H 6735 1710 50  0001 C CNN
+F 4 "0402" H 6560 1710 50  0000 R CNN "display_footprint"
+F 5 "6.3V" H 6560 1610 50  0000 R CNN "Voltage"
+F 6 "X5R" H 6560 1510 50  0000 R CNN "Dielectric"
+F 7 "490-13211-1-ND" H 6710 1610 50  0001 C CNN "Digi-Key PN"
+F 8 "WIFI" H 6550 1780 50  0000 R CNN "Configuration"
+	1    6710 1610
+	1    0    0    -1
+$EndComp
+$Comp
+L Custom_Library:C_Custom C?
+U 1 1 6020F910
+P 7410 1610
+AR Path="/5CB7718D/6020F910" Ref="C?"  Part="1"
+AR Path="/5E0DC082/6020F910" Ref="C?"  Part="1"
+AR Path="/5E0F9110/6020F910" Ref="C?"  Part="1"
+AR Path="/5A557C58/6020F910" Ref="C?"  Part="1"
+AR Path="/5CB25152/6020F910" Ref="C?"  Part="1"
+AR Path="/5E697934/6020F910" Ref="C?"  Part="1"
+AR Path="/5EAE2F02/6020F910" Ref="C?"  Part="1"
+AR Path="/5EAE3021/6020F910" Ref="C?"  Part="1"
+AR Path="/5EAE2D8A/6020F910" Ref="C?"  Part="1"
+AR Path="/5F581B64/6020F910" Ref="C?"  Part="1"
+AR Path="/5F582E44/6020F910" Ref="C?"  Part="1"
+F 0 "C?" H 7435 1710 50  0000 L CNN
+F 1 "10uF" H 7435 1510 50  0000 L CNN
+F 2 "Capacitors_SMD:C_0402" H 7448 1460 50  0001 C CNN
+F 3 "" H 7435 1710 50  0001 C CNN
+F 4 "0402" H 7260 1710 50  0000 R CNN "display_footprint"
+F 5 "6.3V" H 7260 1610 50  0000 R CNN "Voltage"
+F 6 "X5R" H 7260 1510 50  0000 R CNN "Dielectric"
+F 7 "490-13211-1-ND" H 7410 1610 50  0001 C CNN "Digi-Key PN"
+F 8 "WIFI" H 7250 1780 50  0000 R CNN "Configuration"
+	1    7410 1610
+	1    0    0    -1
+$EndComp
+$Comp
+L Custom_Library:R_Custom R?
+U 1 1 5FF2C483
+P 7330 2930
+AR Path="/5D6B2673/5FF2C483" Ref="R?"  Part="1"
+AR Path="/5D6C0D23/5FF2C483" Ref="R?"  Part="1"
+AR Path="/5D77A516/5FF2C483" Ref="R?"  Part="1"
+AR Path="/5E939CFF/5FF2C483" Ref="R?"  Part="1"
+AR Path="/5F581B41/5FF2C483" Ref="R?"  Part="1"
+AR Path="/5F582E44/5FF2C483" Ref="R?"  Part="1"
+F 0 "R?" H 7240 2930 50  0000 R CNN
+F 1 "10k" V 7330 2860 50  0000 L CNN
+F 2 "Resistors_SMD:R_0402" H 7330 2930 50  0001 C CNN
+F 3 "" H 7330 2930 50  0001 C CNN
+F 4 "0402" H 7430 3000 50  0000 L CNN "display_footprint"
+F 5 "1%" H 7430 2900 50  0000 L CNN "Tolerance"
+F 6 "1/16W" H 7430 2800 50  0000 L CNN "Wattage"
+F 7 "" H 7630 3330 60  0001 C CNN "Digi-Key PN"
+	1    7330 2930
+	-1   0    0    -1
 $EndComp
 $EndSCHEMATC

Commit message: more schematic progress
Parts:
- added C?: 0.1uF, Capacitors_SMD:C_0402, symbol Custom_Library:C_Custom
- added D?: Green, LEDs:LED_0603, symbol Device:LED
- added R?: 1k, Resistors_SMD:R_0603, symbol Custom_Library:R_Custom
- added U?: 74LVC1G97, Package_TO_SOT_SMD:SOT-363_SC-70-6, symbol Custom_Library:74LVC1G97_Power_BUF
- U?: footprint (none) -> Custom Footprints Library:XCVR_ATWINC1500-MR210PB
Connections:
- net +3V3: now also C?.1, R?.1, U?.5 (VCC)
- net GND: now also U?.12 (GND), U?.28 (GND), C?.2, U?.2 (GND), U?.3 (GND), U?.6 (GND)
- net ~WIFI_SPI_SS: now also U?.1
- new net: D?.1 (K), U?.4
- new net: D?.2 (A), R?.2
- no-connect marks 0 -> 5
Changed lines of the file:
@@
 F 0 "U?" H 5650 5151 50  0000 L BNN
 F 1 "ATWINC1500-MR210PB" H 5649 2198 50  0000 L BNN
-F 2 "" H 6250 3700 50  0001 L BNN
+F 2 "Custom Footprints Library:XCVR_ATWINC1500-MR210PB" H 6250 3700 50  0001 L BNN
 F 3 "https://ww1.microchip.com/downloads/en/DeviceDoc/ATWINC15x0-MR210xB-IEEE-802.11-b-g-n-SmartConnect-IoT-Module-Data-Sheet-DS70005304C.pdf" H 6250 3700 50  0001 L BNN
 F 4 "ATWINC1500-MR210PB-ND" H 6250 3700 50  0001 C CNN "Digi-Key PN"
@@
 	-1   0    0    -1
 $EndComp
+Wire Wire Line
+	7000 4800 7080 4800
+Wire Wire Line
+	7080 4800 7080 4900
+Connection ~ 7080 4900
+Wire Wire Line
+	7000 4700 7080 4700
+Wire Wire Line
+	7080 4700 7080 4800
+Connection ~ 7080 4800
+NoConn ~ 5500 4000
+NoConn ~ 5500 4100
+NoConn ~ 5500 4200
+NoConn ~ 5500 4300
+NoConn ~ 5500 4400
+$Comp
+L Custom_Library:C_Custom C?
+U 1 1 601C0E29
+P 2630 6480
+AR Path="/5BAAE1F3/601C0E29" Ref="C?"  Part="1"
+AR Path="/5BAAE1CB/601C0E29" Ref="C?"  Part="1"
+AR Path="/5BE48F98/601C0E29" Ref="C?"  Part="1"
+AR Path="/5CAD2D97/601C0E29" Ref="C?"  Part="1"
+AR Path="/5CB7A8BC/601C0E29" Ref="C?"  Part="1"
+AR Path="/5E6AF016/601C0E29" Ref="C?"  Part="1"
+AR Path="/5EAE4AE4/601C0E29" Ref="C?"  Part="1"
+AR Path="/5F582E50/601C0E29" Ref="C?"  Part="1"
+AR Path="/5F5829C2/601C0E29" Ref="C?"  Part="1"
+AR Path="/5F582E44/601C0E29" Ref="C?"  Part="1"
+F 0 "C?" H 2655 6580 50  0000 L CNN
+F 1 "0.1uF" H 2655 6380 50  0000 L CNN
+F 2 "Capacitors_SMD:C_0402" H 2668 6330 50  0001 C CNN
+F 3 "" H 2655 6580 50  0001 C CNN
+F 4 "490-10701-1-ND" H 3055 6980 60  0001 C CNN "Digi-Key PN"
+F 5 "0402" H 2480 6580 50  0000 R CNN "display_footprint"
+F 6 "50V" H 2480 6480 50  0000 R CNN "Voltage"
+F 7 "X7R" H 2480 6380 50  0000 R CNN "Dielectric"
+	1    2630 6480
+	-1   0    0    -1
+$EndComp
+$Comp
+L power:+3.3V #PWR?
+U 1 1 601C0E2F
+P 2630 6330
+AR Path="/5F582E50/601C0E2F" Ref="#PWR?"  Part="1"
+AR Path="/5F5829C2/601C0E2F" Ref="#PWR?"  Part="1"
+AR Path="/5F582E44/601C0E2F" Ref="#PWR?"  Part="1"
+F 0 "#PWR?" H 2630 6180 50  0001 C CNN
+F 1 "+3.3V" H 2630 6470 50  0000 C CNN
+F 2 "" H 2630 6330 50  0001 C CNN
+F 3 "" H 2630 6330 50  0001 C CNN
+	1    2630 6330
+	1    0    0    -1
+$EndComp
+$Comp
+L power:GND #PWR?
+U 1 1 601C0E35
+P 2630 6630
+AR Path="/5F582E50/601C0E35" Ref="#PWR?"  Part="1"
+AR Path="/5F5829C2/601C0E35" Ref="#PWR?"  Part="1"
+AR Path="/5F582E44/601C0E35" Ref="#PWR?"  Part="1"
+F 0 "#PWR?" H 2630 6380 50  0001 C CNN
+F 1 "GND" H 2630 6480 50  0000 C CNN
+F 2 "" H 2630 6630 50  0001 C CNN
+F 3 "" H 2630 6630 50  0001 C CNN
+	1    2630 6630
+	1    0    0    -1
+$EndComp
+$Comp
+L power:+3.3V #PWR?
+U 1 1 601C0E3B
+P 2740 7070
+AR Path="/5F582E50/601C0E3B" Ref="#PWR?"  Part="1"
+AR Path="/5F5829C2/601C0E3B" Ref="#PWR?"  Part="1"
+AR Path="/5F582E44/601C0E3B" Ref="#PWR?"  Part="1"
+F 0 "#PWR?" H 2740 6920 50  0001 C CNN
+F 1 "+3.3V" H 2740 7210 50  0000 C CNN
+F 2 "" H 2740 7070 50  0001 C CNN
+F 3 "" H 2740 7070 50  0001 C CNN
+	1    2740 7070
+	1    0    0    -1
+$EndComp
+$Comp
+L power:GND #PWR?
+U 1 1 601C0E41
+P 2740 7270
+AR Path="/5F582E50/601C0E41" Ref="#PWR?"  Part="1"
+AR Path="/5F5829C2/601C0E41" Ref="#PWR?"  Part="1"
+AR Path="/5F582E44/601C0E41" Ref="#PWR?"  Part="1"
+F 0 "#PWR?" H 2740 7020 50  0001 C CNN
+F 1 "GND" H 2740 7120 50  0000 C CNN
+F 2 "" H 2740 7270 50  0001 C CNN
+F 3 "" H 2740 7270 50  0001 C CNN
+	1    2740 7270
+	1    0    0    -1
+$EndComp
+$Comp
+L Custom_Library:74LVC1G97_Power_BUF U?
+U 1 1 601C0E47
+P 2740 7170
+AR Path="/5F5829C2/601C0E47" Ref="U?"  Part="1"
+AR Path="/5F582E44/601C0E47" Ref="U?"  Part="1"
+F 0 "U?" H 2800 7320 50  0000 L CNN
+F 1 "74LVC1G97" H 2800 7020 50  0000 L CNN
+F 2 "Package_TO_SOT_SMD:SOT-363_SC-70-6" H 2790 7170 50  0001 C CNN
+F 3 "http://www.ti.com/lit/ds/symlink/sn74lvc1g97.pdf" H 2790 7170 50  0001 C CNN
+	1    2740 7170
+	1    0    0    -1
+$EndComp
+Text GLabel 2440 7170 0    40   Input ~ 0
+~WIFI_SPI_SS
+$Comp
+L Device:LED D?
+U 1 1 601C5578
+P 3310 6900
+AR Path="/5BB844FD/601C5578" Ref="D?"  Part="1"
+AR Path="/5BF346B3/601C5578" Ref="D?"  Part="1"
+AR Path="/5BAAE1F3/601C5578" Ref="D?"  Part="1"
+AR Path="/5CAD2D97/601C5578" Ref="D?"  Part="1"
+AR Path="/5CB7A8BC/601C5578" Ref="D?"  Part="1"
+AR Path="/5CB7A8C3/601C5578" Ref="D?"  Part="1"
+AR Path="/5E93CC4E/601C5578" Ref="D?"  Part="1"
+AR Path="/5F582E4A/601C5578" Ref="D?"  Part="1"
+F 0 "D?" V 3349 6783 50  0000 R CNN
+F 1 "Green" V 3258 6783 50  0000 R CNN
+F 2 "LEDs:LED_0603" H 3310 6900 50  0001 C CNN
+F 3 "~" H 3310 6900 50  0001 C CNN
+F 4 "754-1121-1-ND" H -1850 580 50  0001 C CNN "Digi-Key PN"
+	1    3310 6900
+	0    -1   -1   0
+$EndComp
+Wire Wire Line
+	2990 7170 3310 7170
+Wire Wire Line
+	3310 7170 3310 7050
+$Comp
+L Custom_Library:R_Custom R?
+U 1 1 601C5584
+P 3310 6600
+AR Path="/5BAAE1F3/601C5584" Ref="R?"  Part="1"
+AR Path="/5BAAE1DC/601C5584" Ref="R?"  Part="1"
+AR Path="/5BAAE16C/601C5584" Ref="R?"  Part="1"
+AR Path="/5BB844FD/601C5584" Ref="R?"  Part="1"
+AR Path="/5BF346B3/601C5584" Ref="R?"  Part="1"
+AR Path="/5CAD2D97/601C5584" Ref="R?"  Part="1"
+AR Path="/5CB7A8BC/601C5584" Ref="R?"  Part="1"
+AR Path="/5CB7A8C3/601C5584" Ref="R?"  Part="1"
+AR Path="/5E93CC4E/601C5584" Ref="R?"  Part="1"
+AR Path="/5F582E4A/601C5584" Ref="R?"  Part="1"
+F 0 "R?" H 3250 6600 50  0000 R CNN
+F 1 "1k" V 3310 6600 50  0000 C CNN
+F 2 "Resistors_SMD:R_0603" H 3310 6600 50  0001 C CNN
+F 3 "" H 3310 6600 50  0001 C CNN
+F 4 "0603" H 3380 6680 50  0000 L CNN "display_footprint"
+F 5 "1%" H 3380 6600 50  0000 L CNN "Tolerance"
+F 6 "1/10W" H 3380 6530 50  0000 L CNN "Wattage"
+F 7 "311-1.00KHRCT-ND" H 3610 7000 60  0001 C CNN "Digi-Key PN"
+	1    3310 6600
+	-1   0    0    -1
+$EndComp
+$Comp
+L power:+3.3V #PWR?
+U 1 1 601C558A
+P 3310 6450
+AR Path="/5CB7A8BC/601C558A" Ref="#PWR?"  Part="1"
+AR Path="/5CB7A8C3/601C558A" Ref="#PWR?"  Part="1"
+AR Path="/5E93CC4E/601C558A" Ref="#PWR?"  Part="1"
+AR Path="/5F582E4A/601C558A" Ref="#PWR?"  Part="1"
+F 0 "#PWR?" H 3310 6300 50  0001 C CNN
+F 1 "+3.3V" H 3310 6590 50  0000 C CNN
+F 2 "" H 3310 6450 50  0001 C CNN
+F 3 "" H 3310 6450 50  0001 C CNN
+	1    3310 6450
+	1    0    0    -1
+$EndComp
 $EndSCHEMATC
