File: hdw/LED_Panel_Controller/WiFi_Module.sch (KiCad schematic (older format))
At the start: 37 parts, among them J1801 WIFI_I2C, U1801 74LVC1G97, U1802 74LVC1G97, U1803 ATWINC1500-MR210PB

Commit message: having a mid-project crisis
Parts:
- removed C1801, C1802: 0.1uF, Capacitors_SMD:C_0402, symbol Custom_Library:C_Custom
- removed C1803, C1804, C1805, C1807, C1808: 10uF, Capacitors_SMD:C_0402, symbol Custom_Library:C_Custom
- removed C1806: 10nF, Capacitors_SMD:C_0402, symbol Custom_Library:C_Custom
- removed D1801, D1802: Green, LEDs:LED_0402, symbol Device:LED
- removed J1801: WIFI_I2C, Connector_PinHeader_2.54mm:PinHeader_1x03_P2.54mm_Vertical, symbol Connector_Generic:Conn_01x03
- removed R1801, R1802, R1803, R1804, R1805, R1806, R1822: 10, Resistors_SMD:R_0402, symbol Custom_Library:R_Custom
- removed R1807, R1808, R1810, R1811, R1813, R1814, R1815, R1816, R1817, R1819, R1820, R1821: 10k, Resistors_SMD:R_0402, symbol Custom_Library:R_Custom
- removed R1809, R1818: 1k, Resistors_SMD:R_0402, symbol Custom_Library:R_Custom
- removed R1812: 1M, Resistors_SMD:R_0402, symbol Custom_Library:R_Custom
- removed TP1801: TP, Custom Footprints Library:Test_Point, symbol Custom_Library:TP_Pad
- removed U1801, U1802: 74LVC1G97, Package_TO_SOT_SMD:SOT-363_SC-70-6, symbol Custom_Library:74LVC1G97_Power_BUF
- removed U1803: ATWINC1500-MR210PB, Custom Footprints Library:XCVR_ATWINC1500-MR210PB, symbol Custom_Library:ATWINC1500-MR210PB
Connections:
- no-connect marks 4 -> 0
