File: hdw/LED_Panel_Controller/LED_Panel_Controller.kicad_pcb (KiCad board)
At the start: 4 copper layers, 100 x 100 mm, 597 parts, among them J1201 PIC_UART, J1202 WIFI_UART, J1203 I2C, J1204 WIFI_SPI, J1205 SD_SPI, J1206 FLASH_SPI, J1501 USB_B_Mini, J1701 Micro_SD_Card_Det_Hirose_DM3AT, J1801 WIFI_I2C, J201 +12V IN, J202 Keystone_8191, J203 Keystone_8191, J3301 Panel Data, J3302 Keystone_8191, J3303 Keystone_8191, J801 PICKIT4, Q401 BSS214NW, Q402 ZXMS6004FFTA, Q601 BSS214NW, Q602 ZXMS6004FFTA, Q801 BSS214NW, SW2201 Cap_Touch, SW2202 Cap_Touch, SW801 MRST, U1001 74LVC1G97, U1101 PIC32MZ2048EFG100_IPF, U1201 MCP9804, U1301 LTC1694, U1302 AT24CS32-STUM, U1401 DS1683, U1501 74LVC1G97, U1502 CP2105, U1503 TXB0104RGY, U1504 TPD3S014DBVR, U1601 INA219BxDCN, U1602 MCP9804, U1701 74LVC1G97, U1702 74LVC1G97, U1801 74LVC1G97, U1802 74LVC1G97, U1803 ATWINC1500-MR210PB, U1901 74LVC1G97, U1902 74LVC1G97, U1903 74LVC1G97, U1904 74LVC1G97, U1905 74LVC1G97, U2001 74LVC1G97, U2002 74LVC1G97, U2003 74LVC1G97, U2004 74LVC1G97, U201 TPS26600RHFT, U2101 DS3231MZ, U2102 TLV6700, U2201 AT42QT1010-TSHR, U2202 AT42QT1010-TSHR, U2203 74LVC1G97, U2204 74LVC1G97, U2301 74LVC1G97, U2302 74LVC1G97, U2303 74LVC1G97, U2304 74LVC1G97, U2305 74LVC1G97, U2306 74LVC1G97, U2307 74LVC1G97, U2308 74LVC1G97, U2401 74LVC1G97, U2402 SST25VF080B-50-4I-S2AF, U2501 74LVC1G97, U2502 SST25VF080B-50-4I-S2AF, U2601 74LVC1G97, U2602 SST25VF080B-50-4I-S2AF, U2701 74LVC1G97, U2702 SST25VF080B-50-4I-S2AF, U2801 74LVC1G97, U2802 SST25VF080B-50-4I-S2AF, U2901 74LVC1G97, U2902 SST25VF080B-50-4I-S2AF, U3001 74LVC1G97, U3002 SST25VF080B-50-4I-S2AF, U301 INA219BxDCN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

Commit message: fixed SPI flash pull resistors, more PCB placement
Parts:
- C801, D801, J3301, Q801, R1101, R1102, R801, R802, R803, R804, R805: moved to B.Cu
- U2402, U2502, U2602, U2702, U2802, U2902, U3002, U3102: value SST25VF080B-50-4I-S2AF -> SST25VF080B
- moved C901 565.9 mm to (119.1, 35.4), turned to 90 degrees
- moved L901 565.7 mm to (124.2, 47.0), turned to 270 degrees
- moved C916 563.1 mm to (126.4, 24.7)
- moved C915 562.8 mm to (126.4, 25.7)
- moved C910 562.2 mm to (124.9, 44.7)
- moved L902 561.4 mm to (125.6, 47.0), turned to 270 degrees
- moved C903 560.5 mm to (118.2, 35.4), turned to 90 degrees
- moved C912 559.4 mm to (124.9, 45.6)
- moved C914 555.6 mm to (130.9, 24.7), turned to 180 degrees
- moved C913 555.3 mm to (130.9, 25.7), turned to 180 degrees
- moved C906 553.2 mm to (127.9, 45.6), turned to 180 degrees
- moved C907 551.7 mm to (132.4, 44.7), turned to 180 degrees
- moved C905 550.4 mm to (127.9, 44.7), turned to 180 degrees
- moved D801 549.4 mm to (84.5, 41.1), turned to 90 degrees
- moved C908 546.0 mm to (132.4, 45.6), turned to 180 degrees
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Connections:
- D801 pad 3: +3V3 -> Net-(D801-Pad3)
- D801 pad 4: PIC32MZ_ICSPDAT -> PIC32MZ_ICSPCLK
- D801 pad 5: PIC32MZ_ICSPCLK -> PIC32MZ_ICSPDAT
- D801 pad 6: Net-(D801-Pad6) -> +3V3
- R2406 pad 2: GND -> +3V3
- R2407 pad 2: GND -> +3V3
- R2408 pad 2: GND -> +3V3
- R2506 pad 2: GND -> +3V3
- R2507 pad 2: GND -> +3V3
- R2508 pad 2: GND -> +3V3
- R2606 pad 2: GND -> +3V3
- R2607 pad 2: GND -> +3V3
- R2608 pad 2: GND -> +3V3
- R2706 pad 2: GND -> +3V3
- R2707 pad 2: GND -> +3V3
- R2708 pad 2: GND -> +3V3
- R2806 pad 2: GND -> +3V3
- R2807 pad 2: GND -> +3V3
- R2808 pad 2: GND -> +3V3
- R2906 pad 2: GND -> +3V3
- R2907 pad 2: GND -> +3V3
- R2908 pad 2: GND -> +3V3
- R3006 pad 2: GND -> +3V3
- R3007 pad 2: GND -> +3V3
- R3008 pad 2: GND -> +3V3
- R3106 pad 2: GND -> +3V3
- R3107 pad 2: GND -> +3V3
- R3108 pad 2: GND -> +3V3
Other:
- board text added: "MCLR"
- board text added: "REFCLK1 (1MHz)"

Commit message: more PCB grouping, fanout optimization
Parts:
- C1704, C301, C302, C303, D1702, D201, R1703, R1704, R1706, R1707, R1708, R201, R2103, R216, R217, R219, R3219, R3220, R3221, R3222, R3223, R3224, R3225, R3226, R3227, R3228, R3229, R3230, R3231, R3232, R3233, R3234, R3235, R3236, R3237, R3238, R3239, R3240, R3241, R3242, R3243, R3244, R3245, R3246, R3247, R3248, U301, U302: moved to B.Cu
- moved C2101 519.3 mm to (118.4, 37.7), turned to 180 degrees
- moved C2104 458.5 mm to (184.8, 53.4), turned to 180 degrees
- moved TP2101 436.0 mm to (176.1, 35.5)
- moved D1401 430.4 mm to (245.1, 24.8), turned to 180 degrees
- moved R2102 428.2 mm to (209.8, 53.6), turned to 90 degrees
- moved U2102 427.0 mm to (212.3, 53.1)
- moved C1403 425.8 mm to (249.2, 24.8), turned to 90 degrees
- moved BT2102 425.6 mm to (193.5, 30.8)
- moved C1401 425.5 mm to (247.2, 24.8), turned to 90 degrees
- moved U1401 421.9 mm to (247.1, 28.9)
- moved C1402 421.5 mm to (248.2, 24.8), turned to 90 degrees
- moved C2102 419.7 mm to (195.6, 55.3), turned to 270 degrees
- moved C2103 417.4 mm to (194.6, 55.3), turned to 270 degrees
- moved C1404 416.5 mm to (250.1, 24.8), turned to 90 degrees
- moved U2101 416.3 mm to (190.0, 54.1)
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Connections:
- D1702 pad 3: SD_SPI_MOSI -> Net-(D1702-Pad3)
- D1702 pad 5: SD_SPI_MISO -> Net-(D1702-Pad5)
- D1702 pad 6: ~SD_CARD_DET_R -> Net-(D1702-Pad6)
- J1701 pad 10: Net-(J1701-Pad10) -> Net-(D1702-Pad3)
- J1701 pad 3: Net-(J1701-Pad3) -> Net-(D1702-Pad6)
- J1701 pad 5: Net-(J1701-Pad5) -> Net-(D1702-Pad5)
- J1701 pad 7: SD_SPI_MISO -> Net-(D1702-Pad4)
- R1702 pad 2: SD_SPI_SCK -> SD_SPI_MISO
- R1706 pad 2: Net-(D1702-Pad4) -> SD_SPI_SCK
- R1709 pad 1: Net-(J1701-Pad3) -> Net-(D1702-Pad6)
- R1710 pad 1: Net-(J1701-Pad5) -> Net-(D1702-Pad5)
- R1710 pad 2: Net-(D1702-Pad4) -> SD_SPI_SCK
- R1711 pad 1: Net-(J1701-Pad10) -> Net-(D1702-Pad3)
Other:
- board text added: "+12V"
- board text added: "+12VIN"
- board text added: "SD Access"

Commit message: more PCB grouping
Parts:
- C1302, C1804, C1807, C1808, C503, R1807, R1808, R1810, R1811, R1813, R1814, R1815, R1816, R1817, R1819, R1820, R1821, R401, R408, R409, R410, U502: moved to B.Cu
- moved C1802 460.5 mm to (24.0, 164.2)
- moved R1816 459.9 mm to (26.7, 161.7)
- moved R1809 457.0 mm to (23.5, 151.2), turned to 180 degrees
- moved C1806 453.9 mm to (26.7, 160.7), turned to 180 degrees
- moved TP1801 453.3 mm to (24.1, 160.7)
- moved R1810 453.1 mm to (26.7, 158.7), turned to 180 degrees
- moved R1807 451.2 mm to (35.1, 170.1), turned to 90 degrees
- moved R1818 450.1 mm to (21.2, 166.4), turned to 180 degrees
- moved C1801 450.1 mm to (26.3, 149.0)
- moved D1801 448.4 mm to (23.5, 150.0), turned to 180 degrees
- moved C1804 447.6 mm to (26.7, 159.7), turned to 180 degrees
- moved R1804 447.2 mm to (36.1, 150.2), turned to 90 degrees
- moved R1819 446.5 mm to (34.1, 170.1), turned to 90 degrees
- moved R1801 446.2 mm to (35.1, 170.1), turned to 270 degrees
- moved C1808 445.7 mm to (26.7, 160.7), turned to 180 degrees
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Other:
- board text added: "+3.3V"
- board text added: "WIFI AUX"
- board text added: "WIFI COM"
- board text added: "WIFI VCORE"

Commit message: USB/power PCB grouping
Parts:
- C1501, C1502, C1503, C1504, C1505, C1506, C1507, C1509, C1510, C1601, C1602, C703, R1507, R1508, R1509, R1510, R1513, R1514, R1515, R1518, R1519, R1520, R1521, R601, R608, R609, R610, U1501, U1502, U1503, U1601, U702: moved to B.Cu
- L401: value 3.3uH -> 2.2uH; footprint Inductors_SMD:L_Vishay_IHLP-1212 -> Inductors_SMD:L_Vishay_IHLP-2020
- U402: value TPS62152 -> TPS62132
- moved R604 417.5 mm to (142.1, 161.3)
- moved C603 416.3 mm to (141.6, 156.7), turned to 180 degrees
- moved Q601 411.8 mm to (142.1, 159.1), turned to 90 degrees
- moved R603 411.2 mm to (143.6, 156.7)
- moved D601 403.4 mm to (139.7, 159.1), turned to 270 degrees
- moved Q602 402.2 mm to (145.4, 159.1)
- moved R605 398.9 mm to (159.6, 153.6), turned to 90 degrees
- moved C605 397.0 mm to (157.7, 156.0), turned to 90 degrees
- moved R602 395.7 mm to (162.8, 153.6), turned to 270 degrees
- moved R613 394.8 mm to (160.6, 153.6), turned to 90 degrees
- moved C604 393.9 mm to (158.6, 153.6), turned to 90 degrees
- moved R609 392.7 mm to (163.8, 164.9), turned to 270 degrees
- moved R601 392.2 mm to (166.7, 149.8), turned to 180 degrees
- moved R606 391.5 mm to (167.8, 164.4), turned to 180 degrees
- moved R612 391.2 mm to (161.7, 153.6), turned to 270 degrees
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Connections:
- R1507 pad 2: WIFI_UART_TX -> WIFI_UART_RX
- R1508 pad 2: WIFI_UART_RX -> WIFI_UART_TX
- R1509 pad 2: PIC32MZ_UART_TX -> PIC32MZ_UART_RX
- R1510 pad 2: PIC32MZ_UART_RX -> PIC32MZ_UART_TX
- R1518 pad 2: PIC32MZ_UART_RX_BUF -> PIC32MZ_UART_TX_BUF
- R1519 pad 2: PIC32MZ_UART_TX_BUF -> PIC32MZ_UART_RX_BUF
- R1520 pad 2: WIFI_UART_RX_BUF -> WIFI_UART_TX_BUF
- R1521 pad 2: WIFI_UART_TX_BUF -> WIFI_UART_RX_BUF
- U1503 pad 10: WIFI_UART_TX_BUF -> WIFI_UART_RX_BUF
- U1503 pad 11: WIFI_UART_RX_BUF -> WIFI_UART_TX_BUF
- U1503 pad 12: PIC32MZ_UART_TX_BUF -> PIC32MZ_UART_RX_BUF
- U1503 pad 13: PIC32MZ_UART_RX_BUF -> PIC32MZ_UART_TX_BUF
- U1503 pad 2: PIC32MZ_UART_RX -> PIC32MZ_UART_TX
- U1503 pad 3: PIC32MZ_UART_TX -> PIC32MZ_UART_RX
- U1503 pad 4: WIFI_UART_RX -> WIFI_UART_TX
- U1503 pad 5: WIFI_UART_TX -> WIFI_UART_RX
Other:
- board text added: "+5V"
- board text added: "+5V_USB"
- board text added: "Host"
- board text added: "RX"
- board text added: "TX"
- board text added: "WiFi"
