File: hdw/LED_Panel_Controller/LED_Panel_Controller.kicad_pcb (KiCad board)
At the start: 4 copper layers, 100 x 100 mm, 597 parts, among them J1201 PIC_UART, J1202 WIFI_UART, J1203 I2C, J1204 WIFI_SPI, J1205 SD_SPI, J1206 FLASH_SPI, J1501 USB_B_Mini, J1701 Micro_SD_Card_Det_Hirose_DM3AT, J1801 WIFI_I2C, J201 +12V IN, J202 Keystone_8191, J203 Keystone_8191, J3301 Panel Data, J3302 Keystone_8191, J3303 Keystone_8191, J801 PICKIT4, Q401 BSS214NW, Q402 ZXMS6004FFTA, Q601 BSS214NW, Q602 ZXMS6004FFTA, Q801 BSS214NW, SW2201 Cap_Touch, SW2202 Cap_Touch, SW801 MRST, U1001 74LVC1G97, U1101 PIC32MZ2048EFG100_IPF, U1201 MCP9804, U1301 LTC1694, U1302 AT24CS32-STUM, U1401 DS1683, U1501 74LVC1G97, U1502 CP2105, U1503 TXB0104RGY, U1504 TPD3S014DBVR, U1601 INA219BxDCN, U1602 MCP9804, U1701 74LVC1G97, U1702 74LVC1G97, U1801 74LVC1G97, U1802 74LVC1G97, U1803 ATWINC1500-MR210PB, U1901 74LVC1G97, U1902 74LVC1G97, U1903 74LVC1G97, U1904 74LVC1G97, U1905 74LVC1G97, U2001 74LVC1G97, U2002 74LVC1G97, U2003 74LVC1G97, U2004 74LVC1G97, U201 TPS26600RHFT, U2101 DS3231MZ, U2102 TLV6700, U2201 AT42QT1010-TSHR, U2202 AT42QT1010-TSHR, U2203 74LVC1G97, U2204 74LVC1G97, U2301 74LVC1G97, U2302 74LVC1G97, U2303 74LVC1G97, U2304 74LVC1G97, U2305 74LVC1G97, U2306 74LVC1G97, U2307 74LVC1G97, U2308 74LVC1G97, U2401 74LVC1G97, U2402 SST25VF080B, U2501 74LVC1G97, U2502 SST25VF080B, U2601 74LVC1G97, U2602 SST25VF080B, U2701 74LVC1G97, U2702 SST25VF080B, U2801 74LVC1G97, U2802 SST25VF080B, U2901 74LVC1G97, U2902 SST25VF080B, U3001 74LVC1G97, U3002 SST25VF080B, U301 INA219BxDCN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

Commit message: LED PCB grouping
Parts:
- R1901, R2001, R2002, R2005, R2006, R2301, R2302, R2303, R2307, R2308, R2309, R2313, R2314: moved to B.Cu
- moved R2002 341.9 mm to (223.2, 84.3), turned to 270 degrees
- moved R2001 338.5 mm to (223.2, 79.2), turned to 270 degrees
- moved R2004 336.5 mm to (226.2, 84.0)
- moved R2007 336.0 mm to (226.2, 89.1)
- moved R2006 334.7 mm to (223.2, 94.5), turned to 270 degrees
- moved D2001 333.8 mm to (226.2, 80.2)
- moved C2003 333.1 mm to (223.2, 91.3), turned to 180 degrees
- moved D2004 332.9 mm to (226.2, 95.4)
- moved C2004 332.7 mm to (223.2, 96.4), turned to 180 degrees
- moved R2003 332.7 mm to (226.2, 78.9)
- moved R2005 332.2 mm to (223.2, 89.4), turned to 270 degrees
- moved C2001 329.9 mm to (223.2, 81.2), turned to 180 degrees
- moved D2002 329.5 mm to (226.2, 85.2)
- moved C2002 329.3 mm to (223.2, 86.3), turned to 180 degrees
- moved U2004 329.2 mm to (223.2, 94.5)
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
Commit message: finished pcb grouping by sheet
Parts:
- C2203, C2204, C2205, C2206, C2207, C2208, C3301, D3301, D3302, D3303, R2202, R2204, R2209, R2210: moved to B.Cu
- moved J1201 345.2 mm to (198.9, 85.9)
- moved J1204 345.2 mm to (180.3, 85.9)
- moved J1205 345.2 mm to (175.6, 85.9)
- moved J1202 345.2 mm to (194.2, 85.9)
- moved J1203 345.2 mm to (189.6, 85.9)
- moved J1206 345.2 mm to (184.9, 85.9)
- moved R2204 220.6 mm to (227.5, 128.3), turned to 270 degrees
- moved R2203 218.3 mm to (227.5, 128.3), turned to 270 degrees
- moved R2205 217.8 mm to (227.5, 139.4), turned to 270 degrees
- moved C2203 217.0 mm to (230.3, 139.8), turned to 180 degrees
- moved R2206 215.6 mm to (227.5, 125.4), turned to 270 degrees
- moved C2207 215.6 mm to (230.3, 135.2)
- moved R2201 215.2 mm to (227.5, 142.2), turned to 270 degrees
- moved R2209 215.0 mm to (230.3, 134.2)
- moved SW2201 214.2 mm to (221.5, 138.1)
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Connections:
- D3301 pad 1: G0_POS5 -> R0_POS5
- D3301 pad 3: R0_POS5 -> G1_POS5
- D3301 pad 5: G1_POS5 -> B0_POS5
- D3301 pad 6: B0_POS5 -> G0_POS5
- D3302 pad 3: Row_E_POS5 -> Row_C_POS5
- D3302 pad 4: Row_D_POS5 -> Row_B_POS5
- D3302 pad 5: Row_B_POS5 -> Row_A_POS5
- D3302 pad 6: Row_A_POS5 -> Row_E_POS5
- D3303 pad 1: Panel_LAT_POS5 -> Row_D_POS5
- D3303 pad 3: Row_C_POS5 -> Net-(D3303-Pad3)
- D3303 pad 4: Panel_CLK_POS5 -> ~Panel_OE_POS5
- D3303 pad 5: Net-(D3303-Pad5) -> Panel_LAT_POS5
- D3303 pad 6: ~Panel_OE_POS5 -> Panel_CLK_POS5
Routing:
- net R0_POS5: track 0.00 -> 10.4 mm
- net B1_POS5: track 0.00 -> 9.18 mm
- net ~Panel_OE_POS5: track 0.00 -> 8.87 mm
- net Row_C_POS5: track 0.00 -> 8.58 mm
- net B0_POS5: track 0.00 -> 6.38 mm
- net R1_POS5: track 0.00 -> 6.15 mm
- net Panel_CLK_POS5: track 0.00 -> 6.03 mm
- net Row_A_POS5: track 0.00 -> 5.90 mm
- net Row_D_POS5: track 0.00 -> 5.88 mm
- net G1_POS5: track 0.00 -> 5.51 mm
- net G0_POS5: track 0.00 -> 3.57 mm
- net Row_B_POS5: track 0.00 -> 3.09 mm
- net Row_E_POS5: track 0.00 -> 3.04 mm
- net Panel_LAT_POS5: track 0.00 -> 2.91 mm
- net GND: track 0.00 -> 2.64 mm

Commit message: established board outline for connector cutout
Parts:
- moved C1801 303.2 mm to (329.2, 135.3)
- moved C1802 303.2 mm to (326.9, 150.5)
- moved C1901 303.2 mm to (551.2, 66.2)
- moved C1902 303.2 mm to (551.2, 71.3)
- moved C1903 303.2 mm to (551.2, 76.4)
- moved C1904 303.2 mm to (551.2, 81.4)
- moved C1905 303.2 mm to (551.2, 86.5)
- moved C203 303.2 mm to (360.9, 102.4)
- moved C2105 303.2 mm to (515.2, 41.8)
- moved C2201 303.2 mm to (533.2, 128.5)
- moved C2202 303.2 mm to (533.2, 114.5)
- moved C2203 303.2 mm to (533.2, 126.1)
- moved C2204 303.2 mm to (533.2, 112.2)
- moved C2205 303.2 mm to (533.2, 123.6)
- moved C2206 303.2 mm to (533.2, 109.6)
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Other:
- outline, holes or cut-outs redrawn

Commit message: optimized panel signal level shifter signal locations
Parts:
- moved R3262 331.2 mm to (85.9, 92.8), turned to 180 degrees
- moved R3261 331.2 mm to (85.9, 93.8), turned to 180 degrees
- moved R3260 331.1 mm to (85.9, 94.8), turned to 180 degrees
- moved R3254 331.0 mm to (86.0, 84.8), turned to 180 degrees
- moved R3259 331.0 mm to (85.9, 95.8), turned to 180 degrees
- moved R3253 331.0 mm to (86.0, 85.9), turned to 180 degrees
- moved R3258 331.0 mm to (85.9, 96.8), turned to 180 degrees
- moved R3257 330.9 mm to (85.9, 97.8), turned to 180 degrees
- moved R3252 330.9 mm to (86.0, 86.9), turned to 180 degrees
- moved R3256 330.9 mm to (85.9, 98.9), turned to 180 degrees
- moved R3255 330.9 mm to (85.9, 99.9), turned to 180 degrees
- moved R3251 330.9 mm to (86.0, 87.9), turned to 180 degrees
- moved R3250 330.8 mm to (86.0, 88.9), turned to 180 degrees
- moved R3249 330.8 mm to (86.0, 89.9), turned to 180 degrees
- moved R3235 323.4 mm to (89.8, 92.8), turned to 0 degrees
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Connections:
- R3201 pad 2: R0_POS3P3 -> B1_POS3P3
- R3202 pad 2: R1_POS3P3 -> G1_POS3P3
- R3203 pad 2: G0_POS3P3 -> R1_POS3P3
- R3204 pad 2: G1_POS3P3 -> B0_POS3P3
- R3205 pad 2: B0_POS3P3 -> G0_POS3P3
- R3206 pad 2: B1_POS3P3 -> R0_POS3P3
- R3207 pad 2: Row_A_POS3P3 -> ~Panel_OE_DIM_POS3P3
- R3208 pad 2: Row_B_POS3P3 -> Panel_LAT_POS3P3
- R3209 pad 2: Row_C_POS3P3 -> Panel_CLK_POS3P3
- R3211 pad 2: Row_E_POS3P3 -> Row_C_POS3P3
- R3212 pad 2: Panel_CLK_POS3P3 -> Row_B_POS3P3
- R3213 pad 2: Panel_LAT_POS3P3 -> Net-(R3213-Pad2)
- R3214 pad 2: ~Panel_OE_DIM_POS3P3 -> Row_E_POS3P3
- R3248 pad 1: Net-(R3248-Pad1) -> +5V
- R3248 pad 2: GND -> Net-(R3248-Pad2)
- R3249 pad 2: R0_POS5 -> B1_POS5
- R3250 pad 2: R1_POS5 -> G1_POS5
- R3251 pad 2: G0_POS5 -> R1_POS5
- R3252 pad 2: G1_POS5 -> B0_POS5
- R3253 pad 2: B0_POS5 -> G0_POS5
- R3254 pad 2: B1_POS5 -> R0_POS5
- R3255 pad 1: Net-(R3248-Pad1) -> Net-(R3248-Pad2)
- R3255 pad 2: Row_A_POS5 -> ~Panel_OE_POS5
- R3256 pad 2: Row_B_POS5 -> Panel_LAT_POS5
- R3257 pad 2: Row_C_POS5 -> Panel_CLK_POS5
- R3259 pad 2: Row_E_POS5 -> Row_C_POS5
- R3260 pad 2: Panel_CLK_POS5 -> Row_B_POS5
- R3261 pad 2: Panel_LAT_POS5 -> Row_A_POS5
- R3262 pad 2: ~Panel_OE_POS5 -> Row_E_POS5
- U3203 pad 18: Net-(R3248-Pad1) -> Net-(R3248-Pad2)
Routing:
- net R0_POS5: track 10.4 -> 18.2 mm
- net B0_POS5: track 6.38 -> 14.0 mm
- net Row_A_POS5: track 5.90 -> 13.1 mm
- net Row_C_POS5: track 8.58 -> 15.6 mm
- net R1_POS5: track 6.15 -> 13.1 mm
- net Panel_CLK_POS5: track 6.03 -> 12.8 mm
- net ~Panel_OE_POS5: track 8.87 -> 15.7 mm
- net B1_POS5: track 9.18 -> 16.0 mm
- net G0_POS5: track 3.57 -> 8.20 mm
- net Row_E_POS5: track 3.04 -> 7.32 mm
- net Row_B_POS5: track 3.09 -> 7.16 mm
- net Row_D_POS5: track 5.88 -> 9.74 mm
- net G1_POS5: track 5.51 -> 9.30 mm
- net Panel_LAT_POS5: track 2.91 -> 6.56 mm

Commit message: arranging major PCB functional blocks
Parts:
- added REF**: Symbol_Barrel_Polarity, Symbol:Symbol_Barrel_Polarity, F.Cu at (97.6, 51.8)
- L1502: moved to B.Cu
- moved C2201 441.9 mm to (91.3, 129.8)
- moved C2202 441.9 mm to (91.3, 115.9)
- moved C2203 441.9 mm to (91.3, 127.5)
- moved C2204 441.9 mm to (91.3, 113.5)
- moved C2205 441.9 mm to (91.3, 125.0)
- moved C2206 441.9 mm to (91.3, 111.0)
- moved C2207 441.9 mm to (91.3, 122.9)
- moved C2208 441.9 mm to (91.3, 109.0)
- moved R2207 441.9 mm to (91.3, 125.0)
- moved R2208 441.9 mm to (91.3, 111.0)
- moved R2209 441.9 mm to (91.3, 121.9)
- moved R2210 441.9 mm to (91.3, 108.0)
- moved SW2201 441.9 mm to (82.5, 125.8)
- moved SW2202 441.9 mm to (82.5, 111.8)
- moved U2201 441.9 mm to (91.3, 127.5)
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Other:
- board text added: "+"
- board text added: "-"
- board text added: "ATWINC I2C"
- board text added: "GND"
- board text added: "GNDIN"
- board text added: "SCL"
- board text added: "SDA"

Commit message: more major PCB functional blocks
Parts:
- C403, C603, D401, D601, Q401, Q402, Q601, Q602, R402, R404, R603, R604: moved to B.Cu
- moved C3302 518.1 mm to (11.4, 81.8)
- moved J3302 518.1 mm to (20.8, 73.1)
- moved J3303 518.1 mm to (10.9, 73.1)
- moved C701 391.4 mm to (90.7, 72.8), turned to 270 degrees
- moved C702 390.8 mm to (93.2, 75.9), turned to 0 degrees
- moved R611 390.5 mm to (89.1, 69.2), turned to 90 degrees
- moved R606 389.3 mm to (90.1, 69.2), turned to 90 degrees
- moved U701 388.9 mm to (93.2, 73.5), turned to 0 degrees
- moved R610 388.4 mm to (89.6, 67.3), turned to 180 degrees
- moved R607 387.6 mm to (89.6, 66.2), turned to 180 degrees
- moved R608 387.6 mm to (89.6, 66.2), turned to 180 degrees
- moved R609 386.8 mm to (89.6, 65.2), turned to 180 degrees
- moved TP601 385.6 mm to (88.8, 62.3), turned to 270 degrees
- moved C607 381.7 mm to (91.7, 61.8), turned to 90 degrees
- moved L601 381.6 mm to (95.2, 67.3), turned to 180 degrees
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
Commit message: PCB function blocks taking shape
Parts:
- removed J3303: Keystone_8191, Custom Footprints Library:Keystone_8191
- moved C1401 503.3 mm to (100.8, 237.9)
- moved U1401 503.3 mm to (100.7, 242.0)
- moved C1402 503.3 mm to (101.8, 237.9)
- moved C1403 503.3 mm to (102.8, 237.9)
- moved D1401 503.3 mm to (98.7, 237.9)
- moved C1404 503.3 mm to (103.7, 237.9)
- moved C1901 490.8 mm to (71.5, 169.9)
- moved C1902 490.8 mm to (71.5, 175.0)
- moved C1903 490.8 mm to (71.5, 180.0)
- moved C1904 490.8 mm to (71.5, 185.1)
- moved C1905 490.8 mm to (71.5, 190.2)
- moved R1901 490.8 mm to (71.5, 167.9)
- moved U1901 490.8 mm to (71.5, 167.9)
- moved U1902 490.8 mm to (71.5, 173.0)
- moved U1903 490.8 mm to (71.5, 178.1)
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Other:
- board text added: "+5VOUT"
- board text added: "GNDIN/OUT"
- board text added: "PICKIT4"
- board text removed: "GNDIN"
