File: hdw/LED_Panel_Controller/I2C_Boost.sch (KiCad schematic (older format))
At the start: 4 parts, among them U1301 LTC1694, U1302 AT24CS32-STUM

Commit message: added BOMs, some consolidation
Parts:
- C1301, C1302: Digi-Key PN 490-10701-1-ND -> 490-10698-1-ND
Changed lines of the file:
@@
 F 5 "50V" H 4190 3780 50  0000 R CNN "Voltage"
 F 6 "X7R" H 4190 3680 50  0000 R CNN "Dielectric"
-F 7 "490-10701-1-ND" H 4765 4280 60  0001 C CNN "Digi-Key PN"
+F 7 "490-10698-1-ND" H 4765 4280 60  0001 C CNN "Digi-Key PN"
 F 8 "DNP" H 4110 3970 50  0000 C CNN "Configuration"
 	1    4340 3780
@@
 F 5 "50V" H 4190 5420 50  0000 R CNN "Voltage"
 F 6 "X7R" H 4190 5320 50  0000 R CNN "Dielectric"
-F 7 "490-10701-1-ND" H 4765 5920 60  0001 C CNN "Digi-Key PN"
+F 7 "490-10698-1-ND" H 4765 5920 60  0001 C CNN "Digi-Key PN"
 F 8 "" H 4110 5610 50  0001 C CNN "Configuration"
 	1    4340 5420
