File: hdw/LED_Panel_Controller/POS3P3_Power_Supply.sch (KiCad schematic (older format))
At the start: 27 parts, among them Q401 BSS214NW, Q402 ZXMS6004FFTA, U401 74LVC1G97, U402 TPS62132

Commit message: added BOMs, some consolidation
Parts:
- C401, C405: Digi-Key PN 490-10701-1-ND -> 490-10698-1-ND
Changed lines of the file:
@@
 F 5 "50V" H 4400 2970 50  0000 R CNN "Voltage"
 F 6 "X7R" H 4400 2870 50  0000 R CNN "Dielectric"
-F 7 "490-10701-1-ND" H 4550 2970 50  0001 C CNN "Digi-Key PN"
+F 7 "490-10698-1-ND" H 4550 2970 50  0001 C CNN "Digi-Key PN"
 	1    4550 2970
 	1    0    0    -1
@@
 F 5 "50V" H 2490 4860 50  0000 R CNN "Voltage"
 F 6 "X7R" H 2490 4760 50  0000 R CNN "Dielectric"
-F 7 "490-10701-1-ND" H 2640 4860 50  0001 C CNN "Digi-Key PN"
+F 7 "490-10698-1-ND" H 2640 4860 50  0001 C CNN "Digi-Key PN"
 	1    2640 4860
 	1    0    0    -1
